File: cartridge/cartridge.sch (KiCad schematic (older format))
At the start: 29 parts, among them SW1 DS01-254-S-02BE, SW2 CL-SB-13B-01T‎, U1 Teensy4.1, U2 SN74CBTLV3126PWR, U3 SST39VF6401B

Commit message: DiscoCart V0.1
Connections:
- net LED is gone; now on net GND: U1.61 (LED)
- net RX+ is gone; now on net GND: U1.60 (R+)
- net RX- is gone; now on net GND: U1.65 (R-)
- net TX+ is gone; now on net GND: U1.63 (T+)
- net TX- is gone; now on net GND: U1.62 (T-)
- net A0: now also U1.11 (9_OUT1C); no longer U1.19 (27_A13_SCK1)
- net A1: now also U1.31 (39_MISO1_OUT1A); no longer U1.20 (28_RX7)
- net A10: now also U1.26 (34_RX8); no longer U1.29 (37_CS)
- net A11: now also U1.18 (26_A12_MOSI1); no longer U1.30 (38_CS1_IN1)
- net A12: now also U1.25 (33_MCLK2); no longer U1.31 (39_MISO1_OUT1A)
- net A13: now also U1.19 (27_A13_SCK1); no longer U1.32 (40_A16)
- net A14: now also U1.20 (28_RX7); no longer U1.33 (41_A17)
- net A15: now also U1.21 (29_TX7); no longer U1.35 (13_SCK_LED)
- net A16: now also U1.10 (8_TX2_IN1); no longer U1.36 (14_A0_TX3_SPDIF_OUT)
- net A17: now also U1.28 (36_CS); no longer U1.37 (15_A1_RX3_SPDIF_IN)
- net A18: now also U1.16 (24_A10_TX6_SCL2); no longer U1.38 (16_A2_RX4_SCL1)
- net A19: now also U1.22 (30_CRX3); no longer U1.39 (17_A3_TX4_SDA1)
- net A2: now also U1.32 (40_A16); no longer U1.21 (29_TX7)
- net A20: now also U1.23 (31_CTX3); no longer U1.40 (18_A4_SDA)
- net A21: now also U1.24 (32_OUT1B); no longer U1.41 (19_A5_SCL)
- net A3: now also U1.12 (10_CS_MQSR); no longer U1.22 (30_CRX3)
- net A4: now also U1.30 (38_CS1_IN1); no longer U1.23 (31_CTX3)
- net A5: now also U1.13 (11_MOSI_CTX1); no longer U1.24 (32_OUT1B)
- net A6: now also U1.29 (37_CS); no longer U1.25 (33_MCLK2)
- net A7: now also U1.14 (12_MISO_MQSL); no longer U1.26 (34_RX8)
- net A9: now also U1.17 (25_A11_RX6_SDA2); no longer U1.28 (36_CS)
- net DQ0: now also U1.5 (3_LRCLK2); no longer U1.2 (0_RX1_CRX2_CS1)
- net DQ1: now also U1.4 (2_OUT2); no longer U1.3 (1_TX1_CTX2_MISO1)
- net DQ10: now also U1.7 (5_IN2); no longer U1.12 (10_CS_MQSR)
- net DQ11: now also U1.6 (4_BCLK2); no longer U1.13 (11_MOSI_CTX1)
- net DQ12: now also U1.37 (15_A1_RX3_SPDIF_IN); no longer U1.14 (12_MISO_MQSL)
- net DQ13: now also U1.36 (14_A0_TX3_SPDIF_OUT); no longer U1.16 (24_A10_TX6_SCL2)
- net DQ14: now also U1.33 (41_A17); no longer U1.17 (25_A11_RX6_SDA2)
- net DQ15: now also U1.35 (13_SCK_LED); no longer U1.18 (26_A12_MOSI1)
- net DQ2: now also U1.3 (1_TX1_CTX2_MISO1); no longer U1.4 (2_OUT2)
- net DQ3: now also U1.2 (0_RX1_CRX2_CS1); no longer U1.5 (3_LRCLK2)
- net DQ4: now also U1.41 (19_A5_SCL); no longer U1.6 (4_BCLK2)
- net DQ5: now also U1.40 (18_A4_SDA); no longer U1.7 (5_IN2)
- net DQ6: now also U1.39 (17_A3_TX4_SDA1); no longer U1.8 (6_OUT1D)
- net DQ7: now also U1.38 (16_A2_RX4_SCL1); no longer U1.9 (7_RX2_OUT1A)
- net DQ8: now also U1.9 (7_RX2_OUT1A); no longer U1.10 (8_TX2_IN1)
- net DQ9: now also U1.8 (6_OUT1D); no longer U1.11 (9_OUT1C)
- net GND: now also U1.50 (VBAT), U1.51 (3V3), U1.52 (GND), U1.53 (PROGRAM), U1.54 (ON_OFF), U1.55 (5V), U1.56 (D-), U1.57 (D+), U1.58 (GND), U1.59 (GND), U1.66 (D-), U1.67 (D+)
- no-connect marks 20 -> 8
Changed lines of the file:
@@
 $Descr A4 11693 8268
 encoding utf-8
-Sheet 1 2
+Sheet 1 1
 Title ""
 Date ""
@@
 Entry Bus Bus
 	6150 6300 6250 6200
+Text Label 1300 2950 2    50   ~ 0
+DQ1
+Text Label 1300 2850 2    50   ~ 0
+DQ2
 Text Label 1300 2750 2    50   ~ 0
-DQ0
-Text Label 1300 2850 2    50   ~ 0
-DQ1
-Text Label 1300 2950 2    50   ~ 0
-DQ2
-Text Label 1300 3050 2    50   ~ 0
 DQ3
+Text Label 3500 3650 0    50   ~ 0
+DQ7
+Text Label 1300 3450 2    50   ~ 0
+DQ8
+Text Label 1300 3350 2    50   ~ 0
+DQ9
+Text Label 1300 3250 2    50   ~ 0
+DQ10
 Text Label 1300 3150 2    50   ~ 0
-DQ4
-Text Label 1300 3250 2    50   ~ 0
-DQ5
-Text Label 1300 3350 2    50   ~ 0
-DQ6
-Text Label 1300 3450 2    50   ~ 0
-DQ7
-Text Label 1300 3550 2    50   ~ 0
-DQ8
-Text Label 1300 3650 2    50   ~ 0
-DQ9
-Text Label 1300 3750 2    50   ~ 0
-DQ10
-Text Label 1300 3850 2    50   ~ 0
 DQ11
-Text Label 1300 4350 2    50   ~ 0
+Text Label 3500 3950 0    50   ~ 0
 DQ15
-Text Label 1300 4250 2    50   ~ 0
+Text Label 3500 4150 0    50   ~ 0
 DQ14
-Text Label 1300 4150 2    50   ~ 0
+Text Label 3500 3850 0    50   ~ 0
 DQ13
-Text Label 1300 3950 2    50   ~ 0
+Text Label 3500 3750 0    50   ~ 0
 DQ12
 $Comp
@@
 Wire Wire Line
 	3500 3950 3800 3950
-Text Label 1300 4450 2    50   ~ 0
+Text Label 1300 3650 2    50   ~ 0
 A0
-Text Label 1300 4550 2    50   ~ 0
+Text Label 3500 4350 0    50   ~ 0
 A1
-Text Label 1300 4650 2    50   ~ 0
+Text Label 3500 4250 0    50   ~ 0
 A2
-Text Label 1300 4750 2    50   ~ 0
+Text Label 1300 3750 2    50   ~ 0
 A3
-Text Label 1300 4850 2    50   ~ 0
+Text Label 3500 4450 0    50   ~ 0
 A4
-Text Label 1300 4950 2    50   ~ 0
+Text Label 1300 3850 2    50   ~ 0
 A5
-Text Label 3500 4950 0    50   ~ 0
+Text Label 3500 4550 0    50   ~ 0
 A6
-Text Label 3500 4850 0    50   ~ 0
+Text Label 1300 3950 2    50   ~ 0
 A7
 Text Label 3500 4750 0    50   ~ 0
 A8
+Text Label 1300 4250 2    50   ~ 0
+A9
+Text Label 3500 4850 0    50   ~ 0
+A10
+Text Label 1300 4350 2    50   ~ 0
+A11
+Text Label 3500 4950 0    50   ~ 0
+A12
+Text Label 1300 4450 2    50   ~ 0
+A13
+Text Label 1300 4550 2    50   ~ 0
+A14
+Text Label 1300 4650 2    50   ~ 0
+A15
+Text Label 1300 3550 2    50   ~ 0
+A16
 Text Label 3500 4650 0    50   ~ 0
-A9
-Text Label 3500 4550 0    50   ~ 0
-A10
-Text Label 3500 4450 0    50   ~ 0
-A11
-Text Label 3500 4350 0    50   ~ 0
-A12
-Text Label 3500 4250 0    50   ~ 0
-A13
-Text Label 3500 4150 0    50   ~ 0
-A14
-Text Label 3500 3950 0    50   ~ 0
-A15
-Text Label 3500 3850 0    50   ~ 0
-A16
-Text Label 3500 3750 0    50   ~ 0
 A17
-Text Label 3500 3650 0    50   ~ 0
+Text Label 1300 4150 2    50   ~ 0
 A18
-Text Label 3500 3550 0    50   ~ 0
+Text Label 1300 4750 2    50   ~ 0
 A19
-Text Label 3500 3450 0    50   ~ 0
+Text Label 1300 4850 2    50   ~ 0
 A20
-Text Label 3500 3350 0    50   ~ 0
-A21
 Wire Wire Line
 	3500 3350 3800 3350
@@
 A[0..21]
 Wire Wire Line
-	1000 2750 1300 2750
-Wire Wire Line
 	1000 2850 1300 2850
 Wire Wire Line
@@
 	1000 3250 1300 3250
 Wire Wire Line
-	1300 3350 1000 3350
-Wire Wire Line
-	1000 3450 1300 3450
-Wire Wire Line
-	1300 3550 1000 3550
-Wire Wire Line
-	1000 3650 1300 3650
-Wire Wire Line
-	1300 3750 1000 3750
-Wire Wire Line
-	1000 3850 1300 3850
-Wire Wire Line
-	1300 3950 1000 3950
-Wire Wire Line
-	1000 4150 1300 4150
-Wire Wire Line
-	1300 4250 1000 4250
-Wire Wire Line
-	1000 4350 1300 4350
-Wire Wire Line
-	1300 4450 1000 4450
-Wire Wire Line
-	1000 4550 1300 4550
-Wire Wire Line
-	1300 4650 1000 4650
-Wire Wire Line
-	1000 4750 1300 4750
+	1000 3350 1300 3350
+Wire Wire Line
+	1300 3450 1000 3450
+Wire Wire Line
+	1000 3550 1300 3550
+Wire Wire Line
+	1300 3650 1000 3650
+Wire Wire Line
+	1000 3750 1300 3750
+Wire Wire Line
+	1300 3850 1000 3850
+Wire Wire Line
+	1000 3950 1300 3950
+Wire Wire Line
+	1300 4150 1000 4150
+Wire Wire Line
+	1000 4250 1300 4250
+Wire Wire Line
+	1300 4350 1000 4350
+Wire Wire Line
+	1000 4450 1300 4450
+Wire Wire Line
+	1300 4550 1000 4550
+Wire Wire Line
+	1000 4650 1300 4650
+Wire Wire Line
+	1300 4750 1000 4750
 Wire Wire Line
 	1300 4850 1000 4850
@@
 Wire Wire Line
 	5800 7250 6100 7250
-NoConn ~ 1300 5150
-NoConn ~ 1300 5250
-NoConn ~ 1300 5400
-NoConn ~ 1300 5500
-NoConn ~ 1300 5600
-NoConn ~ 1300 5700
-NoConn ~ 1300 5800
-NoConn ~ 2100 6100
-NoConn ~ 2250 6100
-NoConn ~ 2400 6100
-NoConn ~ 2550 6100
-NoConn ~ 2700 6100
-Text GLabel 3500 5200 2    50   Input ~ 0
-RX-
-Text GLabel 3500 5300 2    50   Input ~ 0
-GND
-Text GLabel 3500 5400 2    50   Input ~ 0
-TX+
-Text GLabel 3500 5500 2    50   Input ~ 0
-TX-
-Text GLabel 3500 5600 2    50   Input ~ 0
-LED
-Text GLabel 3500 5700 2    50   Input ~ 0
-RX+
-$Sheet
-S 2050 1150 1900 700
-U 614E8D8C
-F0 "ethernet" 50
-F1 "ethernet.sch" 50
-$EndSheet
 $Comp
 L VSmile:D_Schottky_x2_KCom_AAK D1
@@
 	0    -1   -1   0
 $EndComp
+Text Label 1300 4950 2    50   ~ 0
+A21
+Text Label 1300 3050 2    50   ~ 0
+DQ0
+Text Label 3500 3550 0    50   ~ 0
+DQ6
+Text Label 3500 3450 0    50   ~ 0
+DQ5
+Text Label 3500 3350 0    50   ~ 0
+DQ4
+Wire Wire Line
+	1000 2750 1300 2750
+Text Label 2400 6100 3    50   ~ 0
+GND
 Wire Bus Line
 	1000 2000 10650 2000
 Wire Bus Line
 	1000 6300 9050 6300
-Wire Bus Line
-	900  4550 900  6200
 Wire Bus Line
 	6800 4400 6800 6200
@@
 	8600 4500 8600 6200
 Wire Bus Line
-	900  2100 900  4250
+	900  2100 900  6200
 Wire Bus Line
 	10750 2100 10750 4600
@@
 Wire Bus Line
 	3900 3450 3900 6200
+Text Label 1300 5150 2    50   ~ 0
+GND
+Text Label 1300 5250 2    50   ~ 0
+GND
+Text Label 1300 5400 2    50   ~ 0
+GND
+Text Label 1300 5500 2    50   ~ 0
+GND
+Text Label 1300 5600 2    50   ~ 0
+GND
+Text Label 1300 5700 2    50   ~ 0
+GND
+Text Label 1300 5800 2    50   ~ 0
+GND
+Text Label 2100 6100 3    50   ~ 0
+GND
+Text Label 2250 6100 3    50   ~ 0
+GND
+Text Label 2550 6100 3    50   ~ 0
+GND
+Text Label 2700 6100 3    50   ~ 0
+GND
+Text Label 3500 5700 0    50   ~ 0
+GND
+Text Label 3500 5600 0    50   ~ 0
+GND
+Text Label 3500 5500 0    50   ~ 0
+GND
+Text Label 3500 5400 0    50   ~ 0
+GND
+Text Label 3500 5300 0    50   ~ 0
+GND
+Text Label 3500 5200 0    50   ~ 0
+GND
 $EndSCHEMATC

Commit message: Final PCB revision for launch
Parts:
- removed C2, C7: 0.1uF, Capacitor_SMD:C_0805_2012Metric_Pad1.18x1.45mm_HandSolder, symbol Device:C
- U2: value SN74CBTLV3126PWR -> SN74CBTLV3125PW
Connections:
- net GND: no longer U2.5 (2A)
- net RAM_CSB: now also U2.9 (3A)
- net RAM_RWB: now also U2.5 (2A); no longer U2.9 (3A)
Changed lines of the file:
@@
 P 5950 1300
 F 0 "U2" H 5950 1825 50  0000 C CNN
-F 1 "SN74CBTLV3126PWR" H 5950 1734 50  0000 C CNN
+F 1 "SN74CBTLV3125PW" H 5950 1734 50  0000 C CNN
 F 2 "Package_SO:TSSOP-14_4.4x5mm_P0.65mm" H 5750 1700 50  0001 C CNN
 F 3 "" H 5750 1700 50  0001 C CNN
@@
 ROM0_1
 Text Label 6300 1500 0    50   ~ 0
-RAM_RWB
+RAM_CSB
 Text Label 5600 1500 2    50   ~ 0
 WE#
 Text Label 5600 1400 2    50   ~ 0
-GND
+RAM_RWB
 Text Label 5600 1200 2    50   ~ 0
 OE#
@@
 	5000 1200 5000 1000
 Wire Wire Line
-	4750 1300 5300 1300
-Wire Wire Line
-	5300 1300 5300 1750
-Wire Wire Line
-	5300 1750 6750 1750
-Wire Wire Line
 	6750 1750 6750 1400
 Wire Wire Line
 	6750 1400 6300 1400
-Connection ~ 5300 1300
-Wire Wire Line
-	5300 1300 5600 1300
 Text Label 10400 4900 0    50   ~ 0
 WE#
@@
 	4900 6650 5300 6650
 $Comp
-L Device:C C2
-U 1 1 612096E8
-P 2850 7100
-F 0 "C2" H 2965 7146 50  0000 L CNN
-F 1 "0.1uF" H 2965 7055 50  0000 L CNN
-F 2 "Capacitor_SMD:C_0805_2012Metric_Pad1.18x1.45mm_HandSolder" H 2888 6950 50  0001 C CNN
-F 3 "~" H 2850 7100 50  0001 C CNN
-	1    2850 7100
-	1    0    0    -1
-$EndComp
-$Comp
 L Device:C C5
 U 1 1 61209B5C
@@
 $EndComp
 $Comp
-L Device:C C7
-U 1 1 6120A475
-P 4500 7100
-F 0 "C7" H 4615 7146 50  0000 L CNN
-F 1 "0.1uF" H 4615 7055 50  0000 L CNN
-F 2 "Capacitor_SMD:C_0805_2012Metric_Pad1.18x1.45mm_HandSolder" H 4538 6950 50  0001 C CNN
-F 3 "~" H 4500 7100 50  0001 C CNN
-	1    4500 7100
-	1    0    0    -1
-$EndComp
-$Comp
 L Device:C C10
 U 1 1 6120A9E9
@@
 Wire Wire Line
 	5300 6950 6100 6950
-Text Label 2550 7250 0    50   ~ 0
-WE#
 Text Label 3350 7250 0    50   ~ 0
 OE#
-Text Label 4200 7250 0    50   ~ 0
-CE#
 Text Label 4950 7250 0    50   ~ 0
 RST#
 Text Label 5800 7250 0    50   ~ 0
 WP#
-Wire Wire Line
-	2550 7250 2850 7250
-Wire Wire Line
-	4200 7250 4500 7250
 Wire Wire Line
 	3350 7250 3700 7250
@@
 Text Label 2400 6100 3    50   ~ 0
 GND
+Text Label 1300 5150 2    50   ~ 0
+GND
+Text Label 1300 5250 2    50   ~ 0
+GND
+Text Label 1300 5400 2    50   ~ 0
+GND
+Text Label 1300 5500 2    50   ~ 0
+GND
+Text Label 1300 5600 2    50   ~ 0
+GND
+Text Label 1300 5700 2    50   ~ 0
+GND
+Text Label 1300 5800 2    50   ~ 0
+GND
+Text Label 2100 6100 3    50   ~ 0
+GND
+Text Label 2250 6100 3    50   ~ 0
+GND
+Text Label 2550 6100 3    50   ~ 0
+GND
+Text Label 2700 6100 3    50   ~ 0
+GND
+Text Label 3500 5700 0    50   ~ 0
+GND
+Text Label 3500 5600 0    50   ~ 0
+GND
+Text Label 3500 5500 0    50   ~ 0
+GND
+Text Label 3500 5400 0    50   ~ 0
+GND
+Text Label 3500 5300 0    50   ~ 0
+GND
+Text Label 3500 5200 0    50   ~ 0
+GND
+Wire Wire Line
+	4750 1300 5200 1300
+Wire Wire Line
+	5200 1750 5200 1300
+Wire Wire Line
+	5200 1750 6750 1750
+Connection ~ 5200 1300
+Wire Wire Line
+	5200 1300 5600 1300
 Wire Bus Line
 	1000 2000 10650 2000
@@
 Wire Bus Line
 	3900 3450 3900 6200
-Text Label 1300 5150 2    50   ~ 0
-GND
-Text Label 1300 5250 2    50   ~ 0
-GND
-Text Label 1300 5400 2    50   ~ 0
-GND
-Text Label 1300 5500 2    50   ~ 0
-GND
-Text Label 1300 5600 2    50   ~ 0
-GND
-Text Label 1300 5700 2    50   ~ 0
-GND
-Text Label 1300 5800 2    50   ~ 0
-GND
-Text Label 2100 6100 3    50   ~ 0
-GND
-Text Label 2250 6100 3    50   ~ 0
-GND
-Text Label 2550 6100 3    50   ~ 0
-GND
-Text Label 2700 6100 3    50   ~ 0
-GND
-Text Label 3500 5700 0    50   ~ 0
-GND
-Text Label 3500 5600 0    50   ~ 0
-GND
-Text Label 3500 5500 0    50   ~ 0
-GND
-Text Label 3500 5400 0    50   ~ 0
-GND
-Text Label 3500 5300 0    50   ~ 0
-GND
-Text Label 3500 5200 0    50   ~ 0
-GND
 $EndSCHEMATC
